Commit message: feat: 优化 ros1

File: dobot_description/urdf/cr12_robot.urdf (robot description, URDF)
Before this commit: robot cr12_robot, 8 links, 7 joints
Joints:
- joint joint2: limit lower=-6.28 upper=6.28 effort=0 velocity=0 -> lower=-3.14 upper=3.14 effort=0 velocity=0; origin xyz=0 0 0 rpy=-1.57079631189374 1.57079631189374 3.14159265358979 -> xyz=0 0 0 rpy=1.5708 1.5708 0
- joint joint4: limit lower=-6.28 upper=6.28 effort=0 velocity=0 -> lower=-3.14 upper=3.14 effort=0 velocity=0; origin xyz=-0.518 0 0.125 rpy=0 0 -1.5707963267949 -> xyz=-0.518 0 0.125 rpy=0 0 -1.5708
- joint joint5: axis 0 0 0.999999999998195 -> 0 0 1; limit lower=-6.28 upper=6.28 effort=0 velocity=0 -> lower=-3.14 upper=3.14 effort=0 velocity=0; origin xyz=0 -0.125 0 rpy=1.5707963267949 0 0 -> xyz=0 -0.125 0 rpy=1.5708 0 0

File: dobot_description/urdf/cr7_robot.urdf (robot description, URDF)
Before this commit: robot cr7_robot, 8 links, 7 joints
Joints:
- joint joint1: axis 0 0 -1 -> 0 0 1; limit lower=-6.28 upper=6.28 effort=0 velocity=0 -> lower=-3.14 upper=3.14 effort=0 velocity=0
- joint joint2: limit lower=-6.28 upper=6.28 effort=0 velocity=0 -> lower=-3.14 upper=3.14 effort=0 velocity=0; origin xyz=0 0 0 rpy=-1.57080420997483 1.57079631189374 -3.14158502419526 -> xyz=0 0 0 rpy=1.5708 1.5708 0
- joint joint4: axis 0 0 0.999999999969965 -> 0 0 1; limit lower=-6.28 upper=6.28 effort=0 velocity=0 -> lower=-3.14 upper=3.14 effort=0 velocity=0; origin xyz=-0.306999999999969 0 0.116 rpy=0 0 -1.57079677671549 -> xyz=-0.306999999999969 0 0.116 rpy=0 0 -1.5708
- joint joint5: axis 0 0 -1 -> 0 0 1; limit lower=-6.28 upper=6.28 effort=0 velocity=0 -> lower=-3.14 upper=3.14 effort=0 velocity=0; origin xyz=0 -0.116 0 rpy=1.5707963267949 0 0 -> xyz=0 -0.116 0 rpy=1.5708 0 0
- joint joint6: axis 0 0 -1 -> 0 0 1; origin xyz=0 0.104999656773681 0 rpy=-1.5707963267949 0 0 -> xyz=0 0.104999656773681 0 rpy=-1.5708 0 0

File: dobot_gazebo/urdf/cr10_robot.xacro (robot description, xacro)
@@ -104,6 +104,6 @@
       xyz="0 0 1" />
     <limit
-      lower="-3.14"
-      upper="3.14"
+      lower="-6.28"
+      upper="6.28"
       effort="300"
       velocity="100" />
@@ -162,6 +162,6 @@
       xyz="0 0 1" />
     <limit
-      lower="-3.14"
-      upper="3.14"
+      lower="-6.28"
+      upper="6.28"
       effort="300"
       velocity="100" />
@@ -220,6 +220,6 @@
       xyz="0 0 1" />
     <limit
-      lower="-2.861"
-      upper="2.861"
+      lower="-2.79"
+      upper="2.79"
       effort="300"
       velocity="100" />
@@ -278,6 +278,6 @@
       xyz="0 0 1" />
     <limit
-      lower="-3.14"
-      upper="3.14"
+      lower="-6.28"
+      upper="6.28"
       effort="300"
       velocity="100" />
@@ -336,6 +336,6 @@
       xyz="0 0 1" />
     <limit
-      lower="-3.14"
-      upper="3.14"
+      lower="-6.28"
+      upper="6.28"
       effort="300"
       velocity="100" />
@@ -399,27 +399,34 @@
       velocity="100" />
   </joint>
- <xacro:macro name="cr10_transmission" params="joint_name">
-     <transmission name="${joint_name}_trans">
-       <type>transmission_interface/SimpleTransmission</type>
-       <joint name="${joint_name}">
-         <!--<hardwareInterface>hardware_interface/PositionJointInterface</hardwareInterface>-->
-         <hardwareInterface>hardware_interface/PositionJointInterface</hardwareInterface>
-       </joint>
-       <actuator name="${joint_name}_motor">
-         <mechanicalReduction>1</mechanicalReduction>
-       </actuator>
-     </transmission>
- </xacro:macro>
- <xacro:cr10_transmission joint_name="joint1"/>
- <xacro:cr10_transmission joint_name="joint2"/>
- <xacro:cr10_transmission joint_name="joint3"/>
- <xacro:cr10_transmission joint_name="joint4"/>
- <xacro:cr10_transmission joint_name="joint5"/>
- <xacro:cr10_transmission joint_name="joint6"/>
- <!-- ros_control plugin -->
+ <!-- Disable physics for all links -->
+  <gazebo reference="base_link">
+    <kinematic>true</kinematic>
+  </gazebo>
+  <gazebo reference="Link1">
+    <kinematic>true</kinematic>
+  </gazebo>
+  <gazebo reference="Link2">
+    <kinematic>true</kinematic>
+  </gazebo>
+  <gazebo reference="Link3">
+    <kinematic>true</kinematic>
+  </gazebo>
+  <gazebo reference="Link4">
+    <kinematic>true</kinematic>
+  </gazebo>
+  <gazebo reference="Link5">
+    <kinematic>true</kinematic>
+  </gazebo>
+  <gazebo reference="Link6">
+    <kinematic>true</kinematic>
+  </gazebo>
+  <!-- JointPoseTrajectory plugin - no physics simulation, direct joint positioning -->
  <gazebo>
-     <plugin name="gazebo_ros_control" filename="libgazebo_ros_control.so">
-         <robotNamespace>/cr10_robot</robotNamespace>
-     </plugin>
- </gazebo>
+    <plugin name="joint_pose_trajectory_plugin" filename="libgazebo_ros_joint_pose_trajectory.so">
+      <topic>/set_joint_trajectory</topic>
+      <updateRate>100</updateRate>
+      <interpolateX>true</interpolateX>
+      <frame_id>Link6</frame_id>
+    </plugin>
+  </gazebo>
 </robot>

File: dobot_gazebo/urdf/cr12_robot.xacro (robot description, xacro)
@@ -158,5 +158,5 @@
     <origin
       xyz="0 0 0"
-      rpy="-1.57079631189374 1.57079631189374 3.14159265358979" />
+      rpy="1.5708 1.5708 0" />
     <parent
       link="Link1" />
@@ -274,5 +274,5 @@
     <origin
       xyz="-0.518 0 0.125"
-      rpy="0 0 -1.5707963267949" />
+      rpy="0 0 -1.5708" />
     <parent
       link="Link3" />
@@ -332,5 +332,5 @@
     <origin
       xyz="0 -0.125 0"
-      rpy="1.5707963267949 0 0" />
+      rpy="1.5708 0 0" />
     <parent
       link="Link4" />
@@ -338,5 +338,5 @@
       link="Link5" />
     <axis
-      xyz="0 0 0.999999999998195" />
+      xyz="0 0 1" />
     <limit
       lower="-6.28"
@@ -403,27 +403,34 @@
       velocity="100" />
   </joint>
- <xacro:macro name="cr12_transmission" params="joint_name">
-     <transmission name="${joint_name}_trans">
-       <type>transmission_interface/SimpleTransmission</type>
-       <joint name="${joint_name}">
-         <!--<hardwareInterface>hardware_interface/PositionJointInterface</hardwareInterface>-->
-         <hardwareInterface>hardware_interface/PositionJointInterface</hardwareInterface>
-       </joint>
-       <actuator name="${joint_name}_motor">
-         <mechanicalReduction>1</mechanicalReduction>
-       </actuator>
-     </transmission>
- </xacro:macro>
- <xacro:cr12_transmission joint_name="joint1"/>
- <xacro:cr12_transmission joint_name="joint2"/>
- <xacro:cr12_transmission joint_name="joint3"/>
- <xacro:cr12_transmission joint_name="joint4"/>
- <xacro:cr12_transmission joint_name="joint5"/>
- <xacro:cr12_transmission joint_name="joint6"/>
- <!-- ros_control plugin -->
+ <!-- Disable physics for all links -->
+  <gazebo reference="base_link">
+    <kinematic>true</kinematic>
+  </gazebo>
+  <gazebo reference="Link1">
+    <kinematic>true</kinematic>
+  </gazebo>
+  <gazebo reference="Link2">
+    <kinematic>true</kinematic>
+  </gazebo>
+  <gazebo reference="Link3">
+    <kinematic>true</kinematic>
+  </gazebo>
+  <gazebo reference="Link4">
+    <kinematic>true</kinematic>
+  </gazebo>
+  <gazebo reference="Link5">
+    <kinematic>true</kinematic>
+  </gazebo>
+  <gazebo reference="Link6">
+    <kinematic>true</kinematic>
+  </gazebo>
+  <!-- JointPoseTrajectory plugin - no physics simulation, direct joint positioning -->
  <gazebo>
-     <plugin name="gazebo_ros_control" filename="libgazebo_ros_control.so">
-         <robotNamespace>/cr12_robot</robotNamespace>
-     </plugin>
- </gazebo>
+    <plugin name="joint_pose_trajectory_plugin" filename="libgazebo_ros_joint_pose_trajectory.so">
+      <topic>/set_joint_trajectory</topic>
+      <updateRate>100</updateRate>
+      <interpolateX>true</interpolateX>
+      <frame_id>Link6</frame_id>
+    </plugin>
+  </gazebo>
 </robot>

File: dobot_gazebo/urdf/cr16_robot.xacro (robot description, xacro)
@@ -104,6 +104,6 @@
       xyz="0 0 1" />
     <limit
-      lower="-3.14"
-      upper="3.14"
+      lower="-6.28"
+      upper="6.28"
       effort="300"
       velocity="100" />
@@ -162,6 +162,6 @@
       xyz="0 0 1" />
     <limit
-      lower="-3.14"
-      upper="3.14"
+      lower="-6.28"
+      upper="6.28"
       effort="300"
       velocity="100" />
@@ -220,6 +220,6 @@
       xyz="0 0 1" />
     <limit
-      lower="-2.86"
-      upper="2.86"
+      lower="-2.79"
+      upper="2.79"
       effort="300"
       velocity="100" />
@@ -278,6 +278,6 @@
       xyz="0 0 1" />
     <limit
-      lower="-3.14"
-      upper="3.14"
+      lower="-6.28"
+      upper="6.28"
       effort="300"
       velocity="100" />
@@ -336,6 +336,6 @@
       xyz="0 0 1" />
     <limit
-      lower="-3.14"
-      upper="3.14"
+      lower="-6.28"
+      upper="6.28"
       effort="300"
       velocity="100" />
@@ -399,27 +399,34 @@
       velocity="100" />
   </joint>
- <xacro:macro name="cr16_transmission" params="joint_name">
-     <transmission name="${joint_name}_trans">
-       <type>transmission_interface/SimpleTransmission</type>
-       <joint name="${joint_name}">
-         <!--<hardwareInterface>hardware_interface/PositionJointInterface</hardwareInterface>-->
-         <hardwareInterface>hardware_interface/PositionJointInterface</hardwareInterface>
-       </joint>
-       <actuator name="${joint_name}_motor">
-         <mechanicalReduction>1</mechanicalReduction>
-       </actuator>
-     </transmission>
- </xacro:macro>
- <xacro:cr16_transmission joint_name="joint1"/>
- <xacro:cr16_transmission joint_name="joint2"/>
- <xacro:cr16_transmission joint_name="joint3"/>
- <xacro:cr16_transmission joint_name="joint4"/>
- <xacro:cr16_transmission joint_name="joint5"/>
- <xacro:cr16_transmission joint_name="joint6"/>
- <!-- ros_control plugin -->
+ <!-- Disable physics for all links -->
+  <gazebo reference="base_link">
+    <kinematic>true</kinematic>
+  </gazebo>
+  <gazebo reference="Link1">
+    <kinematic>true</kinematic>
+  </gazebo>
+  <gazebo reference="Link2">
+    <kinematic>true</kinematic>
+  </gazebo>
+  <gazebo reference="Link3">
+    <kinematic>true</kinematic>
+  </gazebo>
+  <gazebo reference="Link4">
+    <kinematic>true</kinematic>
+  </gazebo>
+  <gazebo reference="Link5">
+    <kinematic>true</kinematic>
+  </gazebo>
+  <gazebo reference="Link6">
+    <kinematic>true</kinematic>
+  </gazebo>
+  <!-- JointPoseTrajectory plugin - no physics simulation, direct joint positioning -->
  <gazebo>
-     <plugin name="gazebo_ros_control" filename="libgazebo_ros_control.so">
-         <robotNamespace>/cr16_robot</robotNamespace>
-     </plugin>
- </gazebo>
+    <plugin name="joint_pose_trajectory_plugin" filename="libgazebo_ros_joint_pose_trajectory.so">
+      <topic>/set_joint_trajectory</topic>
+      <updateRate>100</updateRate>
+      <interpolateX>true</interpolateX>
+      <frame_id>Link6</frame_id>
+    </plugin>
+  </gazebo>
 </robot>

File: dobot_gazebo/urdf/cr3_robot.xacro (robot description, xacro)
@@ -104,6 +104,6 @@
       xyz="0 0 1" />
     <limit
-      lower="-3.14"
-      upper="3.14"
+      lower="-6.28"
+      upper="6.28"
       effort="300"
       velocity="100" />
@@ -162,6 +162,6 @@
       xyz="0 0 1" />
     <limit
-      lower="-3.14"
-      upper="3.14"
+      lower="-6.28"
+      upper="6.28"
       effort="300"
       velocity="100" />
@@ -220,6 +220,6 @@
       xyz="0 0 1" />
     <limit
-      lower="-2.86"
-      upper="2.86"
+      lower="-2.705"
+      upper="2.705"
       effort="300"
       velocity="100" />
@@ -278,6 +278,6 @@
       xyz="0 0 1" />
     <limit
-      lower="-3.14"
-      upper="3.14"
+      lower="-6.28"
+      upper="6.28"
       effort="300"
       velocity="100" />
@@ -336,6 +336,6 @@
       xyz="0 0 1" />
     <limit
-      lower="-3.14"
-      upper="3.14"
+      lower="-6.28"
+      upper="6.28"
       effort="300"
       velocity="100" />
@@ -399,27 +399,34 @@
       velocity="100" />
   </joint>
- <xacro:macro name="cr3_transmission" params="joint_name">
-     <transmission name="${joint_name}_trans">
-       <type>transmission_interface/SimpleTransmission</type>
-       <joint name="${joint_name}">
-         <!--<hardwareInterface>hardware_interface/PositionJointInterface</hardwareInterface>-->
-         <hardwareInterface>hardware_interface/PositionJointInterface</hardwareInterface>
-       </joint>
-       <actuator name="${joint_name}_motor">
-         <mechanicalReduction>1</mechanicalReduction>
-       </actuator>
-     </transmission>
- </xacro:macro>
- <xacro:cr3_transmission joint_name="joint1"/>
- <xacro:cr3_transmission joint_name="joint2"/>
- <xacro:cr3_transmission joint_name="joint3"/>
- <xacro:cr3_transmission joint_name="joint4"/>
- <xacro:cr3_transmission joint_name="joint5"/>
- <xacro:cr3_transmission joint_name="joint6"/>
- <!-- ros_control plugin -->
+ <!-- Disable physics for all links -->
+  <gazebo reference="base_link">
+    <kinematic>true</kinematic>
+  </gazebo>
+  <gazebo reference="Link1">
+    <kinematic>true</kinematic>
+  </gazebo>
+  <gazebo reference="Link2">
+    <kinematic>true</kinematic>
+  </gazebo>
+  <gazebo reference="Link3">
+    <kinematic>true</kinematic>
+  </gazebo>
+  <gazebo reference="Link4">
+    <kinematic>true</kinematic>
+  </gazebo>
+  <gazebo reference="Link5">
+    <kinematic>true</kinematic>
+  </gazebo>
+  <gazebo reference="Link6">
+    <kinematic>true</kinematic>
+  </gazebo>
+  <!-- JointPoseTrajectory plugin - no physics simulation, direct joint positioning -->
  <gazebo>
-     <plugin name="gazebo_ros_control" filename="libgazebo_ros_control.so">
-         <robotNamespace>/cr3_robot</robotNamespace>
-     </plugin>
- </gazebo>
+    <plugin name="joint_pose_trajectory_plugin" filename="libgazebo_ros_joint_pose_trajectory.so">
+      <topic>/set_joint_trajectory</topic>
+      <updateRate>100</updateRate>
+      <interpolateX>true</interpolateX>
+      <frame_id>Link6</frame_id>
+    </plugin>
+  </gazebo>
 </robot>

File: dobot_gazebo/urdf/cr5_robot.xacro (robot description, xacro)
@@ -74,5 +74,5 @@
     <child link="Link1" />
     <axis xyz="0 0 1" />
-    <limit lower="-3.14" upper="3.14" effort="300" velocity="100" />
+    <limit lower="-6.28" upper="6.28" effort="300" velocity="100" />
   </joint>
   <link name="Link2">
@@ -110,5 +110,5 @@
     <child  link="Link2" />
     <axis xyz="0 0 1" />
-    <limit lower="-3.14" upper="3.14" effort="300" velocity="100" />
+    <limit lower="-6.28" upper="6.28" effort="300" velocity="100" />
   </joint>
   <link name="Link3">
@@ -146,5 +146,5 @@
     <child link="Link3" />
     <axis  xyz="0 0 1" />
-    <limit lower="-2.86"  upper="2.86"  effort="300" velocity="100" />
+    <limit lower="-2.79"  upper="2.79"  effort="300" velocity="100" />
   </joint>
   <link name="Link4">
@@ -181,5 +181,5 @@
     <child link="Link4" />
     <axis xyz="0 0 1" />
-    <limit lower="-3.14" upper="3.14" effort="300" velocity="100" />
+    <limit lower="-6.28" upper="6.28" effort="300" velocity="100" />
   </joint>
   <link
@@ -217,5 +217,5 @@
     <child link="Link5" />
     <axis xyz="0 0 1" />
-    <limit lower="-3.14" upper="3.14" effort="300" velocity="100" />
+    <limit lower="-6.28" upper="6.28" effort="300" velocity="100" />
   </joint>
   <link name="Link6">
@@ -254,27 +254,34 @@
     <limit lower="-6.28" upper="6.28" effort="300" velocity="100" />
   </joint>
- <xacro:macro name="cr5_transmission" params="joint_name">
-     <transmission name="${joint_name}_trans">
-       <type>transmission_interface/SimpleTransmission</type>
-       <joint name="${joint_name}">
-         <!--<hardwareInterface>hardware_interface/PositionJointInterface</hardwareInterface>-->
-         <hardwareInterface>hardware_interface/PositionJointInterface</hardwareInterface>
-       </joint>
-       <actuator name="${joint_name}_motor">
-         <mechanicalReduction>1</mechanicalReduction>
-       </actuator>
-     </transmission>
- </xacro:macro>
- <xacro:cr5_transmission joint_name="joint1"/>
- <xacro:cr5_transmission joint_name="joint2"/>
- <xacro:cr5_transmission joint_name="joint3"/>
- <xacro:cr5_transmission joint_name="joint4"/>
- <xacro:cr5_transmission joint_name="joint5"/>
- <xacro:cr5_transmission joint_name="joint6"/>
- <!-- ros_control plugin -->
+ <!-- Disable physics for all links -->
+  <gazebo reference="base_link">
+    <kinematic>true</kinematic>
+  </gazebo>
+  <gazebo reference="Link1">
+    <kinematic>true</kinematic>
+  </gazebo>
+  <gazebo reference="Link2">
+    <kinematic>true</kinematic>
+  </gazebo>
+  <gazebo reference="Link3">
+    <kinematic>true</kinematic>
+  </gazebo>
+  <gazebo reference="Link4">
+    <kinematic>true</kinematic>
+  </gazebo>
+  <gazebo reference="Link5">
+    <kinematic>true</kinematic>
+  </gazebo>
+  <gazebo reference="Link6">
+    <kinematic>true</kinematic>
+  </gazebo>
+  <!-- JointPoseTrajectory plugin - no physics simulation, direct joint positioning -->
  <gazebo>
-     <plugin name="gazebo_ros_control" filename="libgazebo_ros_control.so">
-         <robotNamespace>/cr5_robot</robotNamespace>
-     </plugin>
- </gazebo>
+    <plugin name="joint_pose_trajectory_plugin" filename="libgazebo_ros_joint_pose_trajectory.so">
+      <topic>/set_joint_trajectory</topic>
+      <updateRate>100</updateRate>
+      <interpolateX>true</interpolateX>
+      <frame_id>Link6</frame_id>
+    </plugin>
+  </gazebo>
 </robot>

File: dobot_gazebo/urdf/cr7_robot.xacro (robot description, xacro)
@@ -105,5 +105,5 @@
       link="Link1" />
     <axis
-      xyz="0 0 -1" />
+      xyz="0 0 1" />
     <limit
       lower="-6.28"
@@ -157,5 +157,5 @@
     <origin
       xyz="0 0 0"
-      rpy="-1.57080420997483 1.57079631189374 -3.14158502419526" />
+      rpy="1.5708 1.5708 0" />
     <parent
       link="Link1" />
@@ -273,5 +273,5 @@
     <origin
       xyz="-0.306999999999969 0 0.116"
-      rpy="0 0 -1.57079677671549" />
+      rpy="0 0 -1.5708" />
     <parent
       link="Link3" />
@@ -279,5 +279,5 @@
       link="Link4" />
     <axis
-      xyz="0 0 0.999999999969965" />
+      xyz="0 0 1" />
     <limit
       lower="-6.28"
@@ -331,5 +331,5 @@
     <origin
       xyz="0 -0.116 0"
-      rpy="1.5707963267949 0 0" />
+      rpy="1.5708 0 0" />
     <parent
       link="Link4" />
@@ -337,5 +337,5 @@
       link="Link5" />
     <axis
-      xyz="0 0 -1" />
+      xyz="0 0 1" />
     <limit
       lower="-6.28"
@@ -389,5 +389,5 @@
     <origin
       xyz="0 0.104999656773681 0"
-      rpy="-1.5707963267949 0 0" />
+      rpy="-1.5708 0 0" />
     <parent
       link="Link5" />
@@ -395,5 +395,5 @@
       link="Link6" />
     <axis
-      xyz="0 0 -1" />
+      xyz="0 0 1" />
     <limit
       lower="-6.28"
@@ -402,27 +402,34 @@
       velocity="100" />
   </joint>
- <xacro:macro name="cr7_transmission" params="joint_name">
-     <transmission name="${joint_name}_trans">
-       <type>transmission_interface/SimpleTransmission</type>
-       <joint name="${joint_name}">
-         <!--<hardwareInterface>hardware_interface/PositionJointInterface</hardwareInterface>-->
-         <hardwareInterface>hardware_interface/PositionJointInterface</hardwareInterface>
-       </joint>
-       <actuator name="${joint_name}_motor">
-         <mechanicalReduction>1</mechanicalReduction>
-       </actuator>
-     </transmission>
- </xacro:macro>
- <xacro:cr7_transmission joint_name="joint1"/>
- <xacro:cr7_transmission joint_name="joint2"/>
- <xacro:cr7_transmission joint_name="joint3"/>
- <xacro:cr7_transmission joint_name="joint4"/>
- <xacro:cr7_transmission joint_name="joint5"/>
- <xacro:cr7_transmission joint_name="joint6"/>
- <!-- ros_control plugin -->
+ <!-- Disable physics for all links -->
+  <gazebo reference="base_link">
+    <kinematic>true</kinematic>
+  </gazebo>
+  <gazebo reference="Link1">
+    <kinematic>true</kinematic>
+  </gazebo>
+  <gazebo reference="Link2">
+    <kinematic>true</kinematic>
+  </gazebo>
+  <gazebo reference="Link3">
+    <kinematic>true</kinematic>
+  </gazebo>
+  <gazebo reference="Link4">
+    <kinematic>true</kinematic>
+  </gazebo>
+  <gazebo reference="Link5">
+    <kinematic>true</kinematic>
+  </gazebo>
+  <gazebo reference="Link6">
+    <kinematic>true</kinematic>
+  </gazebo>
+  <!-- JointPoseTrajectory plugin - no physics simulation, direct joint positioning -->
  <gazebo>
-     <plugin name="gazebo_ros_control" filename="libgazebo_ros_control.so">
-         <robotNamespace>/cr7_robot</robotNamespace>
-     </plugin>
- </gazebo>
+    <plugin name="joint_pose_trajectory_plugin" filename="libgazebo_ros_joint_pose_trajectory.so">
+      <topic>/set_joint_trajectory</topic>
+      <updateRate>100</updateRate>
+      <interpolateX>true</interpolateX>
+      <frame_id>Link6</frame_id>
+    </plugin>
+  </gazebo>
 </robot>

File: dobot_gazebo/urdf/me6_robot.xacro (robot description, xacro)
@@ -55,5 +55,5 @@
         <child link="Link1" />
         <axis xyz="0 0 1" />
-        <limit lower="-6.28" upper="6.28" effort="300" velocity="300" />
+        <limit lower="-6.283" upper="6.283" effort="300" velocity="300" />
     </joint>
     <link name="Link2">
@@ -200,5 +200,5 @@
         <child link="Link6" />
         <axis xyz="0 0 1" />
-        <limit lower="-6.28" upper="6.28" effort="300" velocity="300" />
+        <limit lower="-6.283" upper="6.283" effort="300" velocity="300" />
     </joint>
    <link name="world" />
@@ -224,9 +224,34 @@
  <xacro:robot_transmission joint_name="joint5"/>
  <xacro:robot_transmission joint_name="joint6"/>
- <!-- ros_control plugin -->
+ <!-- Disable physics for all links -->
+  <gazebo reference="base_link">
+    <kinematic>true</kinematic>
+  </gazebo>
+  <gazebo reference="Link1">
+    <kinematic>true</kinematic>
+  </gazebo>
+  <gazebo reference="Link2">
+    <kinematic>true</kinematic>
+  </gazebo>
+  <gazebo reference="Link3">
+    <kinematic>true</kinematic>
+  </gazebo>
+  <gazebo reference="Link4">
+    <kinematic>true</kinematic>
+  </gazebo>
+  <gazebo reference="Link5">
+    <kinematic>true</kinematic>
+  </gazebo>
+  <gazebo reference="Link6">
+    <kinematic>true</kinematic>
+  </gazebo>
+  <!-- JointPoseTrajectory plugin - no physics simulation, direct joint positioning -->
  <gazebo>
-     <plugin name="gazebo_ros_control" filename="libgazebo_ros_control.so">
-         <robotNamespace>/me6_robot</robotNamespace>
-     </plugin>
- </gazebo>
+    <plugin name="joint_pose_trajectory_plugin" filename="libgazebo_ros_joint_pose_trajectory.so">
+      <topic>/set_joint_trajectory</topic>
+      <updateRate>100</updateRate>
+      <interpolateX>true</interpolateX>
+      <frame_id>Link6</frame_id>
+    </plugin>
+  </gazebo>
 </robot>
