Commit message: feat: 优化 ros1

File: dobot_gazebo/urdf/nova2_robot.xacro (robot description, xacro)
@@ -58,5 +58,5 @@
         <parent link="base_link" />
         <child link="Link1" />
-        <axis xyz="0 0 -1" />
+        <axis xyz="0 0 1" />
         <limit lower="-6.28" upper="6.28" effort="300" velocity="100" />
     </joint>
@@ -88,5 +88,5 @@
         <child link="Link2" />
         <axis xyz="0 0 1" />
-        <limit lower="-3.14" upper="3.14" effort="300" velocity="100" />
+        <limit lower="-2.618" upper="2.618" effort="300" velocity="100" />
     </joint>
     <link name="Link3">
@@ -117,5 +117,5 @@
         <child link="Link3" />
         <axis xyz="0 0 1" />
-        <limit lower="-2.79" upper="2.79" effort="300" velocity="100" />
+        <limit lower="-2.618" upper="2.618" effort="300" velocity="100" />
     </joint>
     <link name="Link4">
@@ -145,5 +145,5 @@
         <parent link="Link3" />
         <child link="Link4" />
-        <axis xyz="0 0 -1" />
+        <axis xyz="0 0 1" />
         <limit lower="-6.28" upper="6.28" effort="300" velocity="100" />
     </joint>
@@ -174,5 +174,5 @@
         <parent link="Link4" />
         <child link="Link5" />
-        <axis xyz="0 0 -1" />
+        <axis xyz="0 0 1" />
         <limit lower="-6.28" upper="6.28" effort="300" velocity="100" />
     </joint>
@@ -228,9 +228,34 @@
  <xacro:robot_transmission joint_name="joint5"/>
  <xacro:robot_transmission joint_name="joint6"/>
- <!-- ros_control plugin -->
+ <!-- Disable physics for all links -->
+  <gazebo reference="base_link">
+    <kinematic>true</kinematic>
+  </gazebo>
+  <gazebo reference="Link1">
+    <kinematic>true</kinematic>
+  </gazebo>
+  <gazebo reference="Link2">
+    <kinematic>true</kinematic>
+  </gazebo>
+  <gazebo reference="Link3">
+    <kinematic>true</kinematic>
+  </gazebo>
+  <gazebo reference="Link4">
+    <kinematic>true</kinematic>
+  </gazebo>
+  <gazebo reference="Link5">
+    <kinematic>true</kinematic>
+  </gazebo>
+  <gazebo reference="Link6">
+    <kinematic>true</kinematic>
+  </gazebo>
+  <!-- JointPoseTrajectory plugin - no physics simulation, direct joint positioning -->
  <gazebo>
-     <plugin name="gazebo_ros_control" filename="libgazebo_ros_control.so">
-         <robotNamespace>/nova2_robot</robotNamespace>
-     </plugin>
- </gazebo>
+    <plugin name="joint_pose_trajectory_plugin" filename="libgazebo_ros_joint_pose_trajectory.so">
+      <topic>/set_joint_trajectory</topic>
+      <updateRate>100</updateRate>
+      <interpolateX>true</interpolateX>
+      <frame_id>Link6</frame_id>
+    </plugin>
+  </gazebo>
 </robot>

File: dobot_gazebo/urdf/nova5_robot.xacro (robot description, xacro)
@@ -102,5 +102,5 @@
       link="Link1" />
     <axis
-      xyz="0 0 -0.999999999999855" />
+      xyz="0 0 1" />
     <limit
       lower="-6.28"
@@ -220,6 +220,6 @@
       xyz="0 0 1" />
     <limit
-      lower="-2.79"
-      upper="2.79"
+      lower="-2.723"
+      upper="2.723"
       effort="300"
       velocity="100" />
@@ -276,5 +276,5 @@
       link="Link4" />
     <axis
-      xyz="0 0 -1" />
+      xyz="0 0 1" />
     <limit
       lower="-6.28"
@@ -421,9 +421,34 @@
  <xacro:robot_transmission joint_name="joint5"/>
  <xacro:robot_transmission joint_name="joint6"/>
- <!-- ros_control plugin -->
+ <!-- Disable physics for all links -->
+  <gazebo reference="base_link">
+    <kinematic>true</kinematic>
+  </gazebo>
+  <gazebo reference="Link1">
+    <kinematic>true</kinematic>
+  </gazebo>
+  <gazebo reference="Link2">
+    <kinematic>true</kinematic>
+  </gazebo>
+  <gazebo reference="Link3">
+    <kinematic>true</kinematic>
+  </gazebo>
+  <gazebo reference="Link4">
+    <kinematic>true</kinematic>
+  </gazebo>
+  <gazebo reference="Link5">
+    <kinematic>true</kinematic>
+  </gazebo>
+  <gazebo reference="Link6">
+    <kinematic>true</kinematic>
+  </gazebo>
+  <!-- JointPoseTrajectory plugin - no physics simulation, direct joint positioning -->
  <gazebo>
-     <plugin name="gazebo_ros_control" filename="libgazebo_ros_control.so">
-         <robotNamespace>/nova5_robot</robotNamespace>
-     </plugin>
- </gazebo>
+    <plugin name="joint_pose_trajectory_plugin" filename="libgazebo_ros_joint_pose_trajectory.so">
+      <topic>/set_joint_trajectory</topic>
+      <updateRate>100</updateRate>
+      <interpolateX>true</interpolateX>
+      <frame_id>Link6</frame_id>
+    </plugin>
+  </gazebo>
 </robot>
